Commit message: Update bot.urdf

File: 3Dmodel/bot.urdf (robot description, URDF)
Before this commit: robot packing_robot_motor_based, 6 links, 5 joints
Links:
- removed link link1_base_axis
- removed link link3_forearm
- removed link link4_wrist
- removed link link5_gripper
- added link link1_shoulder_mount; collision box size=0.125 0.125 0.04
- added link link4_whristarm; collision box size=0.041 0.033 0.155
- added link link5_hand; collision box size=0.078 0.026 0.06
- added link link6_greaper; collision box size=0.02 0.065 0.02
- link base_link: geometry collision box size=0.125 0.125 0.09
- link link2_upper_arm: geometry collision box size=0.0485 0.045 0.12
Joints:
- removed joint joint3_elbow
- removed joint joint4_wrist
- removed joint joint5_gripper_rotation
- added joint joint4_whrist: type revolute, parent link2_upper_arm, child link4_whristarm, origin xyz=0 0 0.12, axis 1 0 0, limit lower=-3.839 upper=3.839 effort=15 velocity=1.5
- added joint joint5_hand: type revolute, parent link4_whristarm, child link5_hand, origin xyz=0 0 0.155, axis 1 0 0, limit lower=-3.839 upper=3.839 effort=12 velocity=1.5
- added joint joint7_greaper: type revolute, parent link5_hand, child link6_greaper, origin xyz=0.025 -0.013 0.06, axis 0 1 0, limit lower=-3.839 upper=3.839 effort=20 velocity=2.0
- joint joint1_base_yaw: axis 0 0 -1 -> 0 0 1; child link1_base_axis -> link1_shoulder_mount; limit lower=0 upper=3.839 effort=20 velocity=2.0 -> lower=-3.839 upper=3.839 effort=20 velocity=2.0; origin xyz=0 0 0.100 rpy=0 0 0 -> xyz=0 0 0.09
- joint joint2_shoulder: axis -1 0 0 -> 1 0 0; origin xyz=0 0 0.043 rpy=0 0 0 -> xyz=0 -0.016 0.04; parent link1_base_axis -> link1_shoulder_mount
