Commit message: Update mybot.urdf

File: 3Dmodel/mybot.urdf (robot description, URDF)
Before this commit: robot packing_robot_corrected, 7 links, 6 joints
Links:
- link link6_greaper: geometry collision box size=0.08 0.065 0.0198
Joints:
- joint joint7_greaper: origin xyz=0 0 0.059 -> xyz=0.06 -0.007 0.059

Commit message: Update mybot.urdf

File: 3Dmodel/mybot.urdf (robot description, URDF)
Before this commit: robot packing_robot_corrected, 7 links, 6 joints
Links:
- removed link link3_forearm
- link base_link: geometry collision box size=0.125 0.125 0.065
- link link1_shoulder_mount: geometry collision box size=0.125 0.125 0.06
- link link2_upper_arm: geometry collision box size=0.0485 0.045 0.12
- link link4_whristarm: geometry collision box size=0.041 0.033 0.155
- link link6_greaper: geometry collision box size=0.02 0.065 0.02
Joints:
- removed joint joint3_elbow
- joint joint1_base_yaw: origin xyz=0 0 0.056 -> xyz=0 0 0.065
- joint joint2_shoulder: origin xyz=0 -0.016 0.025 -> xyz=0 -0.016 0.06
- joint joint4_whrist: axis 0 0 1 -> 1 0 0; limit lower=-3.14 upper=3.14 effort=20 velocity=2.0 -> lower=-1.57 upper=1.57 effort=15 velocity=1.5; origin xyz=0 0 0.153 -> xyz=0 0 0.12; parent link3_forearm -> link2_upper_arm
- joint joint5_hand: origin xyz=0 0 0.023 -> xyz=0 0 0.155
- joint joint7_greaper: origin xyz=0.06 -0.007 0.059 -> xyz=0.06 -0.013 0.065

Commit message: Update mybot.urdf

File: 3Dmodel/mybot.urdf (robot description, URDF)
Before this commit: robot packing_robot_corrected, 7 links, 6 joints
Links:
- removed link link1_shoulder_mount
- removed link link2_upper_arm
- removed link link3_forearm
- removed link link4_whristarm
- removed link link5_hand
- removed link link6_greaper
- added link link1_base_to_shoulder; collision box size=0.040 0.040 0.040; visual box size=0.040 0.040 0.040
- added link link23_shoulder_to_elbow; collision box size=0.025 0.025 0.120; visual box size=0.025 0.025 0.120
- added link link45_elbow_to_wrist; collision box size=0.022 0.022 0.160; visual box size=0.022 0.022 0.160
- added link link6_wrist_to_gripper_joint; collision box size=0.020 0.020 0.060; visual box size=0.020 0.020 0.060
- added link link7_gripper_tcp; collision box size=0.015 0.015 0.060; visual box size=0.015 0.015 0.060
- link base_link: geometry collision box size=0.080 0.080 0.095; visual box size=0.080 0.080 0.095
Joints:
- removed joint joint1_base_yaw
- removed joint joint2_shoulder
- removed joint joint3_elbow
- removed joint joint4_whrist
- removed joint joint5_hand
- removed joint joint7_greaper
- added joint joint1_base_yaw_id1: type revolute, parent base_link, child link1_base_to_shoulder, origin xyz=0 0 0.095 rpy=0 0 0, axis 0 0 1, limit lower=-1.919862 upper=1.919862 effort=20 velocity=2.0
- added joint joint23_shoulder_pair_id2_id3: type revolute, parent link1_base_to_shoulder, child link23_shoulder_to_elbow, origin xyz=0 0 0.040 rpy=0 0 0, axis 1 0 0, limit lower=-1.570796 upper=1.570796 effort=15 velocity=1.5
- added joint joint45_elbow_pair_id4_id5: type revolute, parent link23_shoulder_to_elbow, child link45_elbow_to_wrist, origin xyz=0 0 0.120 rpy=0 0 0, axis 1 0 0, limit lower=0.000000 upper=1.919862 effort=15 velocity=1.5
- added joint joint6_wrist_id6: type revolute, parent link45_elbow_to_wrist, child link6_wrist_to_gripper_joint, origin xyz=0 0 0.160 rpy=0 0 0, axis 1 0 0, limit lower=-1.919862 upper=1.919862 effort=12 velocity=1.5
- added joint joint7_gripper_rotation_id7: type revolute, parent link6_wrist_to_gripper_joint, child link7_gripper_tcp, origin xyz=0 0 0.060 rpy=0 0 0, axis 0 1 0, limit lower=-1.919862 upper=1.919862 effort=20 velocity=2.0

Commit message: Update mybot.urdf

File: 3Dmodel/mybot.urdf (robot description, URDF)
Before this commit: robot packing_robot_corrected, 6 links, 5 joints
Links:
- removed link link4_whristarm
- removed link link5_hand
- removed link link6_greaper
- added link link45_forearm, mass 0.54; collision box size=0.041 0.033 0.230; visual box size=0.041 0.033 0.230
- added link link6_wrist, mass 0.08; collision box size=0.078 0.026 0.133; visual box size=0.078 0.026 0.133
- added link link7_gripper, mass 0.03; collision box size=0.02 0.065 0.02; visual box size=0.02 0.065 0.02
- link base_link: mass None -> 0.32; geometry collision box size=0.125 0.125 0.065; visual box size=0.125 0.125 0.065
- link link1_shoulder_mount: mass None -> 0.39; geometry collision box size=0.125 0.125 0.04; visual box size=0.125 0.125 0.04
- link link2_upper_arm: mass None -> 0.31; geometry collision box size=0.0485 0.045 0.171; visual box size=0.0485 0.045 0.171
Joints:
- removed joint joint1_base_yaw
- removed joint joint2_shoulder
- removed joint joint4_whrist
- removed joint joint5_hand
- removed joint joint7_greaper
- added joint joint1_base_yaw_id1: type revolute, parent base_link, child link1_shoulder_mount, origin xyz=0 0 0.065, axis 0 0 1, limit lower=-3.14159 upper=3.14159 effort=20 velocity=2.0
- added joint joint23_shoulder_pair_id2_id3: type revolute, parent link1_shoulder_mount, child link2_upper_arm, origin xyz=0 -0.016 0.04, axis 1 0 0, limit lower=-1.5708 upper=1.5708 effort=15 velocity=1.5
- added joint joint45_elbow_pair_id4_id5: type revolute, parent link2_upper_arm, child link45_forearm, origin xyz=0 0 0.171, axis 1 0 0, limit lower=-1.5708 upper=1.5708 effort=15 velocity=1.5
- added joint joint6_wrist_id6: type revolute, parent link45_forearm, child link6_wrist, origin xyz=0 0 0.230, axis 1 0 0, limit lower=-2.6 upper=2.6 effort=12 velocity=1.5
- added joint joint7_gripper_rotation_id7: type revolute, parent link6_wrist, child link7_gripper, origin xyz=0.025 -0.013 0.133, axis 0 1 0, limit lower=-3.14159 upper=3.14159 effort=20 velocity=2.0
